File: version1/ice header adapter pcb.kicad_sch (KiCad schematic)
At the start: 14 parts, among them P1 TST, P2 TST, P3 TST, P4 TST

Commit message: weiter am pc
Parts:
- removed SAM10-1.27: PINHEAD_PINHD-2X5, Arduino_Wifi_shield_v018_tG:PINHEAD_2X05_127, symbol ice-header-adapter-pcb-rescue:PINHEAD_PINHD-2X5PASSO127
- removed SAM10-2: 87758-1016, con-molex:87758-1016, symbol ice-header-adapter-pcb-rescue:ML10
- removed SAM20-2: 87758-2016, con-molex:87758-2016, symbol ice-header-adapter-pcb-rescue:ML20
- removed SAM20-2.54: ML20, con-harting-ml:ML20, symbol ice-header-adapter-pcb-rescue:ML20
- added Avr1: JTAG, con-harting-ml:ML10, symbol ice-header-adapter-pcb-rescue:ML10
- added J1: FTDI 232, Connector_PinSocket_2.54mm:PinSocket_1x06_P2.54mm_Vertical, symbol Connector_Generic:Conn_01x06
- added JP1: FTDI_VCC, Connector_PinSocket_2.54mm:PinSocket_1x02_P2.54mm_Vertical, symbol Jumper:Jumper_2_Open
- added SW1: Reset, Button_Switch_THT:SW_PUSH_6mm_H5mm, symbol Switch:SW_Push
- renumbered AVR10-2.54 to AVR10-2.1, AVR10-UPDI to AVR10-UPDI1, AVR6-2.54 to AVR6-2.1
Connections:
- net GND: now also Avr1.10, Avr1.2, J1.6 (Pin_6), SW1.2
- net NSRST: now also Avr1.6
- net NTRST: now also Avr1.8
- net TCK: now also Avr1.1
- net TDI: now also Avr1.9
- net TDO: now also Avr1.3
- net TMS: now also Avr1.5
- net VTG: now also Avr1.4, JP1.1 (A)
- net RX: now reaches AVR10-UPDI1.3
- net RX: now also J1.2 (Pin_2)
- net TX: now reaches AVR10-UPDI1.4
- net TX: now also J1.3 (Pin_3)
- net RESET: now reaches AVR10-UPDI1.5
- net RESET: now also SW1.1
- new net VCC: J1.4 (Pin_4), JP1.2 (B)
- no-connect marks 21 -> 13
Other:
- note added: "Debug"
- note added: "RXD1"
- note added: "TXD1"
- note removed: "Also for SWD Table 4-4"
- note removed: "SAM JTAG/SWD Connectors"
- note removed: "Table 4-1"
